Commit message: Add files via upload

File: youbot_description/robots/youbot.urdf.xacro (robot description, xacro)
@@ -21,4 +21,5 @@
   <xacro:include filename="$(find youbot_description)/urdf/materials.urdf.xacro" />
   <xacro:include filename="$(find youbot_description)/urdf/misc/camera_tower.urdf.xacro"/>
+  <xacro:include filename="$(find youbot_description)/urdf/misc/camera_tower_down.urdf.xacro"/>
   <!-- sensors -->
   <xacro:include filename="$(find youbot_description)/urdf/sensors/hokuyo_urg04_laser.urdf.xacro"/>
@@ -33,7 +34,7 @@
   <!-- foot for arm-->
   <xacro:youbot_base name="base"/>
-  <xacro:youbot_plate name="plate" parent="base_link">
-    <origin xyz="-0.159 0 0.046" rpy="0 0 0" />
-  </xacro:youbot_plate>
+  <xacro:camera_tower_down name="camera_tower_down" parent="base_link">
+    <origin xyz="-0.159 0 0.02" rpy="0 0 0" />
+  </xacro:camera_tower_down>
   <xacro:youbot_arm name="arm" parent="base_link">
     <origin xyz="0.143 0 0.046" rpy="0 0 0" />
@@ -54,5 +55,5 @@
   </joint>
    <xacro:camera_tower name="camera_tower" parent="base_link">
-    <origin xyz="-0.29 0.0 0.06" rpy="0 0 0" />
+    <origin xyz="-0.159 0.0 0.04" rpy="0 0 0" />
   </xacro:camera_tower>
   <xacro:property name="camera_link" value="0.05" /> <!-- Size of square 'camera' box -->
